File: Fuente.sch (EAGLE design)
At the start: 1 part, among them IC1 MEGA8-AI

Commit message: Last
Parts:
- added ISP1: AVRISP-6, adafruit:AVRISP-6
Changed lines of the file:
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@@
 <layer number="48" name="Document" color="7" fill="1" visible="no" active="no"/>
 <layer number="49" name="Reference" color="7" fill="1" visible="no" active="no"/>
+<layer number="50" name="dxf" color="7" fill="1" visible="no" active="no"/>
 <layer number="51" name="tDocu" color="6" fill="9" visible="no" active="no"/>
 <layer number="52" name="bDocu" color="7" fill="1" visible="no" active="no"/>
+<layer number="53" name="tGND_GNDA" color="7" fill="9" visible="no" active="no"/>
+<layer number="54" name="bGND_GNDA" color="1" fill="9" visible="no" active="no"/>
+<layer number="56" name="wert" color="7" fill="1" visible="no" active="no"/>
 <layer number="91" name="Nets" color="2" fill="1" visible="yes" active="yes"/>
 <layer number="92" name="Busses" color="1" fill="1" visible="yes" active="yes"/>
@@
 <layer number="97" name="Info" color="7" fill="1" visible="yes" active="yes"/>
 <layer number="98" name="Guide" color="6" fill="1" visible="yes" active="yes"/>
+<layer number="100" name="Muster" color="7" fill="1" visible="no" active="no"/>
+<layer number="101" name="Patch_Top" color="12" fill="4" visible="yes" active="yes"/>
+<layer number="102" name="Vscore" color="7" fill="1" visible="yes" active="yes"/>
+<layer number="103" name="fp3" color="7" fill="1" visible="no" active="yes"/>
+<layer number="104" name="Name" color="7" fill="1" visible="yes" active="yes"/>
+<layer number="105" name="Beschreib" color="9" fill="1" visible="yes" active="yes"/>
+<layer number="106" name="BGA-Top" color="4" fill="1" visible="yes" active="yes"/>
+<layer number="107" name="BD-Top" color="5" fill="1" visible="yes" active="yes"/>
+<layer number="108" name="fp8" color="7" fill="1" visible="no" active="yes"/>
+<layer number="109" name="fp9" color="7" fill="1" visible="no" active="yes"/>
+<layer number="110" name="fp0" color="7" fill="1" visible="no" active="yes"/>
+<layer number="111" name="LPC17xx" color="7" fill="1" visible="yes" active="yes"/>
+<layer number="112" name="tSilk" color="7" fill="1" visible="yes" active="yes"/>
+<layer number="116" name="Patch_BOT" color="9" fill="4" visible="yes" active="yes"/>
+<layer number="121" name="_tsilk" color="7" fill="1" visible="yes" active="yes"/>
+<layer number="122" name="_bsilk" color="7" fill="1" visible="yes" active="yes"/>
+<layer number="123" name="tTestmark" color="7" fill="1" visible="no" active="yes"/>
+<layer number="124" name="bTestmark" color="7" fill="1" visible="no" active="yes"/>
+<layer number="125" name="_tNames" color="7" fill="1" visible="yes" active="yes"/>
+<layer number="126" name="_bNames" color="7" fill="1" visible="yes" active="yes"/>
+<layer number="127" name="_tValues" color="7" fill="1" visible="yes" active="yes"/>
+<layer number="128" name="_bValues" color="7" fill="1" visible="yes" active="yes"/>
+<layer number="131" name="tAdjust" color="7" fill="1" visible="no" active="yes"/>
+<layer number="132" name="bAdjust" color="7" fill="1" visible="no" active="yes"/>
+<layer number="144" name="Drill_legend" color="7" fill="1" visible="yes" active="yes"/>
+<layer number="151" name="HeatSink" color="7" fill="1" visible="yes" active="yes"/>
+<layer number="152" name="_bDocu" color="7" fill="1" visible="yes" active="yes"/>
+<layer number="199" name="Contour" color="7" fill="1" visible="yes" active="yes"/>
+<layer number="200" name="200bmp" color="1" fill="10" visible="yes" active="yes"/>
+<layer number="201" name="201bmp" color="2" fill="1" visible="no" active="no"/>
+<layer number="202" name="202bmp" color="3" fill="1" visible="no" active="no"/>
+<layer number="203" name="203bmp" color="4" fill="10" visible="yes" active="yes"/>
+<layer number="204" name="204bmp" color="5" fill="10" visible="yes" active="yes"/>
+<layer number="205" name="205bmp" color="6" fill="10" visible="yes" active="yes"/>
+<layer number="206" name="206bmp" color="7" fill="10" visible="yes" active="yes"/>
+<layer number="207" name="207bmp" color="8" fill="10" visible="yes" active="yes"/>
+<layer number="208" name="208bmp" color="9" fill="10" visible="yes" active="yes"/>
+<layer number="209" name="209bmp" color="7" fill="1" visible="no" active="yes"/>
+<layer number="210" name="210bmp" color="7" fill="1" visible="no" active="yes"/>
+<layer number="211" name="211bmp" color="7" fill="1" visible="yes" active="yes"/>
+<layer number="212" name="212bmp" color="7" fill="1" visible="yes" active="yes"/>
+<layer number="213" name="213bmp" color="7" fill="1" visible="yes" active="yes"/>
+<layer number="214" name="214bmp" color="7" fill="1" visible="yes" active="yes"/>
+<layer number="215" name="215bmp" color="7" fill="1" visible="yes" active="yes"/>
+<layer number="216" name="216bmp" color="7" fill="1" visible="yes" active="yes"/>
+<layer number="217" name="217bmp" color="18" fill="1" visible="no" active="no"/>
+<layer number="218" name="218bmp" color="19" fill="1" visible="no" active="no"/>
+<layer number="219" name="219bmp" color="20" fill="1" visible="no" active="no"/>
+<layer number="220" name="220bmp" color="21" fill="1" visible="no" active="no"/>
+<layer number="221" name="221bmp" color="22" fill="1" visible="no" active="no"/>
+<layer number="222" name="222bmp" color="23" fill="1" visible="no" active="no"/>
+<layer number="223" name="223bmp" color="24" fill="1" visible="no" active="no"/>
+<layer number="224" name="224bmp" color="25" fill="1" visible="no" active="no"/>
+<layer number="248" name="Housing" color="7" fill="1" visible="yes" active="yes"/>
+<layer number="249" name="Edge" color="7" fill="1" visible="yes" active="yes"/>
+<layer number="250" name="Descript" color="7" fill="1" visible="no" active="no"/>
+<layer number="251" name="SMDround" color="7" fill="1" visible="no" active="no"/>
+<layer number="254" name="cooling" color="7" fill="1" visible="yes" active="yes"/>
 </layers>
 <schematic xreflabel="%F%N/%S.%C%R" xrefpart="/%S.%C%R">
@@
 <parts>
 <part name="IC1" library="atmel" deviceset="MEGA8" device="-AI"/>
+<part name="ISP1" library="adafruit" deviceset="AVRISP" device="-6"/>
 </parts>
 <sheets>
@@
 <instances>
 <instance part="IC1" gate="G$1" x="22.86" y="60.96"/>
+<instance part="ISP1" gate="G$1" x="104.14" y="66.04"/>
 </instances>
 <busses>

Commit message: actu
Parts:
- removed IC1: MEGA8-AI, atmel:MEGA8-AI
- added JP1: USBSMD, SparkFun-Connectors:USBSMD
- added U$1: ATMEGA32U4TQFP, SparkFun-DigitalIC:ATMEGA32U4TQFP
Connections:
- new net MISO: ISP1.MISO, U$1.PB3(MISO)
- new net MOSI: ISP1.MOSI, U$1.PB2(MOSI)
- new net N$3: ISP1.RST
- new net N$4: ISP1.VCC
- new net N$6: ISP1.GND
- new net SCK: ISP1.SCK, U$1.PB1(SCK)
Other:
- moved on the sheet: ISP1
Changed lines of the file:
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@@
 <?xml version="1.0" encoding="utf-8"?>
 <!DOCTYPE eagle SYSTEM "eagle.dtd">
-<eagle version="6.2">
+<eagle version="6.3">
 <drawing>
 <settings>
@@
 </classes>
 <parts>
-<part name="IC1" library="atmel" deviceset="MEGA8" device="-AI"/>
 <part name="ISP1" library="adafruit" deviceset="AVRISP" device="-6"/>
+<part name="U$1" library="SparkFun-DigitalIC" deviceset="ATMEGA32U4" device="TQFP"/>
+<part name="JP1" library="SparkFun-Connectors" deviceset="USB" device="SMD"/>
 </parts>
 <sheets>
@@
 </plain>
 <instances>
-<instance part="IC1" gate="G$1" x="22.86" y="60.96"/>
-<instance part="ISP1" gate="G$1" x="104.14" y="66.04"/>
+<instance part="ISP1" gate="G$1" x="99.06" y="91.44"/>
+<instance part="U$1" gate="G$1" x="17.78" y="58.42"/>
+<instance part="JP1" gate="G$1" x="-38.1" y="71.12" rot="R180"/>
 </instances>
 <busses>
 </busses>
 <nets>
+<net name="MISO" class="0">
+<segment>
+<pinref part="ISP1" gate="G$1" pin="MISO"/>
+<wire x1="86.36" y1="93.98" x2="76.2" y2="93.98" width="0.1524" layer="91"/>
+<label x="78.74" y="93.98" size="1.778" layer="95"/>
+</segment>
+<segment>
+<pinref part="U$1" gate="G$1" pin="PB3(MISO)"/>
+<wire x1="35.56" y1="27.94" x2="45.72" y2="27.94" width="0.1524" layer="91"/>
+<label x="38.1" y="27.94" size="1.778" layer="95"/>
+</segment>
+</net>
+<net name="SCK" class="0">
+<segment>
+<pinref part="ISP1" gate="G$1" pin="SCK"/>
+<wire x1="86.36" y1="91.44" x2="76.2" y2="91.44" width="0.1524" layer="91"/>
+<label x="78.74" y="91.44" size="1.778" layer="95"/>
+</segment>
+<segment>
+<pinref part="U$1" gate="G$1" pin="PB1(SCK)"/>
+<wire x1="35.56" y1="33.02" x2="45.72" y2="33.02" width="0.1524" layer="91"/>
+<label x="38.1" y="33.02" size="1.778" layer="95"/>
+</segment>
+</net>
+<net name="N$3" class="0">
+<segment>
+<pinref part="ISP1" gate="G$1" pin="RST"/>
+<wire x1="86.36" y1="88.9" x2="76.2" y2="88.9" width="0.1524" layer="91"/>
+</segment>
+</net>
+<net name="N$4" class="0">
+<segment>
+<pinref part="ISP1" gate="G$1" pin="VCC"/>
+<wire x1="114.3" y1="93.98" x2="124.46" y2="93.98" width="0.1524" layer="91"/>
+</segment>
+</net>
+<net name="MOSI" class="0">
+<segment>
+<pinref part="ISP1" gate="G$1" pin="MOSI"/>
+<wire x1="114.3" y1="91.44" x2="124.46" y2="91.44" width="0.1524" layer="91"/>
+<label x="119.38" y="91.44" size="1.778" layer="95"/>
+</segment>
+<segment>
+<pinref part="U$1" gate="G$1" pin="PB2(MOSI)"/>
+<wire x1="35.56" y1="30.48" x2="45.72" y2="30.48" width="0.1524" layer="91"/>
+<label x="38.1" y="30.48" size="1.778" layer="95"/>
+</segment>
+</net>
+<net name="N$6" class="0">
+<segment>
+<pinref part="ISP1" gate="G$1" pin="GND"/>
+<wire x1="114.3" y1="88.9" x2="124.46" y2="88.9" width="0.1524" layer="91"/>
+</segment>
+</net>
 </nets>
 </sheet>

Commit message: Sch updated
Parts:
- added C1: 10uF, SparkFun-Capacitors:CAP_POLPTH2
- added F1, F2: (no value), adafruit:PTCFUSE-1812
- added Q1: (no value), SparkFun-DiscreteSemi:TRANSISTOR_NPNSOT23
- added R1, R2, R7, R9: 10k, adafruit:R-US_M0805
- added R10, R11, R12: 220, SparkFun-Resistors:RESISTOR0805-RES
- added R3, R4: .1, adafruit:R-US_R2512
- added R5, R6: 22, adafruit:R-US_0309/12
- added R8: 1k, adafruit:R-US_M0805
- added S1, S5: 50-2POLE30, switch:50-2POLE30
- added S2: 75CF36-2, switch:75CF36-2
- added S3: (no value), switch:CK102X06
- added S4, S6: ELMA-01-2X6, switch:ELMA-01-2X6
- added S7, S8: SWITCH-MOMENTARY-212MM, SparkFun-Electromechanical:SWITCH-MOMENTARY-212MM
- added U$2, U$3: (no value), SparkFun-Electromechanical:POT-RV16AF-20
- added U$4: LED-TRICOLOR, SparkFun-LED:LED-TRICOLOR
- added U1, U2: (no value), microbuilder:INA219
- added Y1: (no value), SparkFun-FreqCtrl:RESONATORPTH
Connections:
- new net 5V: ISP1.VCC, R1.2, R2.2, R7.2, U$1.AVCC@24, U$1.AVCC@44, U$1.UVCC, U$1.VCC@14, U$1.VCC@34, U$4.A, U1.VCC, U2.VCC
- new net GND: C1.-, ISP1.GND, JP1.GND, R9.2, S7.2, U$1.GND@15, U$1.GND@23, U$1.GND@35, U$1.GND@43, U$1.UGND, U1.GND, U2.GND, Y1.2
- new net N$1: R4.2, U2.VIN+
- new net N$10: R6.2, U$1.D-
- new net N$11: JP1.D-, R6.1
- new net N$12: U$1.XTAL1, Y1.1
- new net N$13: U$1.XTAL2, Y1.3
- new net N$14: R11.2, U$4.BLU
- new net N$15: R12.2, U$4.GRN
- new net N$2: F2.1, R4.1, U2.VIN-
- new net N$5: R3.2, U1.VIN+
- new net N$7: F1.1, R3.1, U1.VIN-
- new net N$8: JP1.D+, R5.1
- new net N$9: R5.2, U$1.D+
- new net R1: ISP1.RST, R7.1, S7.1, U$1.!RESET
- new net SCL: R2.1, U$1.PD0(SCL), U1.SCL, U2.SCL
- new net SDA: R1.1, U$1.PD1(SDA), U1.SDA, U2.SDA
- net N$3: now also C1.+, JP1.VBUS, U$1.VBUS; no longer ISP1.RST
- net N$4: now also R9.1, U$1.PE2/!HWB; no longer ISP1.VCC
- net N$6: now also R10.2, U$4.RED; no longer ISP1.GND

Commit message: Sch and Pcb updated
Parts:
- removed S1, S5: 50-2POLE30, switch:50-2POLE30
- removed S2: 75CF36-2, switch:75CF36-2
- removed S3: (no value), switch:CK102X06
- removed S4, S6: ELMA-01-2X6, switch:ELMA-01-2X6
- added JP2, JP3: (no value), SparkFun-Connectors:M08LONGPADS
- added JP4, JP5: (no value), SparkFun-Connectors:M02LOCK_LONGPADS
- added R13, R14, R15, R16: 10k, adafruit:R-US_M0805
Connections:
- removed net N$1: R4.2, U2.VIN+
- removed net N$5: R3.2, U1.VIN+
- new net INV12: JP2.7, JP2.8, JP3.8
- new net INV33: JP2.3, JP2.4, JP3.6
- new net INV5: JP2.5, JP2.6, JP3.7
- new net N$16: F1.2, JP4.2
- new net N$17: F2.2, JP5.2
- new net N$19: JP3.4
- new net N$20: JP3.5
- new net N$28: R13.1, U1.A0
- new net N$29: R14.1, U1.A1
- new net N$30: R15.1, U2.A0
- new net N$31: R16.1, U2.A1
- new net V1: JP2.1, R3.2, U1.VIN+
- new net V2: JP2.2, R4.2, U2.VIN+
- net 5V: now also JP3.3
- net GND: now also JP3.1, JP3.2, JP4.1, JP5.1
Other:
- moved on the sheet: Q1, R10, R11, R12, R8, U$2, U$3, U$4

Commit message: pcb and sch updated
Parts:
- removed R15, R16: 10k, adafruit:R-US_M0805
- R13, R14: value 10k -> 1M
- U$2: value (none) -> M08X2; device SparkFun-Electromechanical:POT-RV16AF-20 -> SparkFun-Connectors:M08X2
Connections:
- removed net N$20: JP3.5
- removed net N$28: R13.1, U1.A0
- removed net N$29: R14.1, U1.A1
- removed net N$30: R15.1, U2.A0
- removed net N$31: R16.1, U2.A1
- new net EN: JP3.5, Q1.C
- new net N$1: Q1.B, R8.1
- new net N$5: ISP1.VCC
- net 5V: no longer ISP1.VCC
- net GND: now also Q1.E, R13.1, R14.1, U1.A0, U1.A1
- net N$2: now also R14.2
- net N$7: now also R13.2
- net SDA: now also U2.A0, U2.A1
Other:
- moved on the sheet: R13, R14, R8
Changed lines of the file:
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@@
 <part name="SUPPLY1" library="SparkFun-Aesthetics" deviceset="5V" device=""/>
 <part name="SUPPLY2" library="SparkFun-Aesthetics" deviceset="5V" device=""/>
-<part name="SUPPLY3" library="SparkFun-Aesthetics" deviceset="5V" device=""/>
 <part name="GND1" library="SparkFun-Aesthetics" deviceset="GND" device=""/>
 <part name="GND2" library="SparkFun-Aesthetics" deviceset="GND" device=""/>
@@
 <part name="GND6" library="SparkFun-Aesthetics" deviceset="GND" device=""/>
 <part name="GND7" library="SparkFun-Aesthetics" deviceset="GND" device=""/>
-<part name="U$2" library="SparkFun-Electromechanical" deviceset="POT" device="-RV16AF-20"/>
 <part name="U$3" library="SparkFun-Electromechanical" deviceset="POT" device="-RV16AF-20"/>
 <part name="U$4" library="SparkFun-LED" deviceset="LED-TRICOLOR" device=""/>
@@
 <part name="JP5" library="SparkFun-Connectors" deviceset="M02" device="LOCK_LONGPADS"/>
 <part name="GND13" library="SparkFun-Aesthetics" deviceset="GND" device=""/>
-<part name="R13" library="adafruit" deviceset="R-US_" device="M0805" value="10k"/>
-<part name="R14" library="adafruit" deviceset="R-US_" device="M0805" value="10k"/>
-<part name="R15" library="adafruit" deviceset="R-US_" device="M0805" value="10k"/>
-<part name="R16" library="adafruit" deviceset="R-US_" device="M0805" value="10k"/>
 <part name="SUPPLY9" library="SparkFun-Aesthetics" deviceset="5V" device=""/>
+<part name="GND8" library="SparkFun-Aesthetics" deviceset="GND" device=""/>
+<part name="GND14" library="SparkFun-Aesthetics" deviceset="GND" device=""/>
+<part name="GND15" library="SparkFun-Aesthetics" deviceset="GND" device=""/>
+<part name="R13" library="adafruit" deviceset="R-US_" device="M0805" value="1M"/>
+<part name="R14" library="adafruit" deviceset="R-US_" device="M0805" value="1M"/>
+<part name="U$2" library="SparkFun-Connectors" deviceset="M08X2" device=""/>
 </parts>
 <sheets>
@@
 <instance part="SUPPLY1" gate="G$1" x="50.8" y="78.74"/>
 <instance part="SUPPLY2" gate="G$1" x="58.42" y="78.74"/>
-<instance part="SUPPLY3" gate="G$1" x="124.46" y="96.52"/>
 <instance part="GND1" gate="1" x="76.2" y="-2.54"/>
 <instance part="GND2" gate="1" x="-2.54" y="15.24"/>
@@
 <instance part="SUPPLY4" gate="G$1" x="-27.94" y="93.98"/>
 <instance part="Q1" gate="G$1" x="-81.28" y="15.24"/>
-<instance part="R8" gate="G$1" x="-66.04" y="15.24" rot="R180"/>
+<instance part="R8" gate="G$1" x="-91.44" y="15.24" rot="R180"/>
 <instance part="F1" gate="G$1" x="124.46" y="40.64"/>
 <instance part="F2" gate="G$1" x="124.46" y="2.54"/>
@@
 <instance part="GND6" gate="1" x="-15.24" y="114.3" rot="R180"/>
 <instance part="GND7" gate="1" x="127" y="83.82"/>
-<instance part="U$2" gate="G$1" x="-40.64" y="12.7" rot="MR0"/>
 <instance part="U$3" gate="G$1" x="-27.94" y="12.7" rot="MR0"/>
 <instance part="U$4" gate="G$1" x="-81.28" y="38.1" rot="MR0"/>
@@
 <instance part="JP5" gate="G$1" x="139.7" y="2.54" rot="MR0"/>
 <instance part="GND13" gate="1" x="132.08" y="-2.54"/>
-<instance part="R13" gate="G$1" x="66.04" y="48.26" rot="R180"/>
-<instance part="R14" gate="G$1" x="66.04" y="40.64" rot="R180"/>
-<instance part="R15" gate="G$1" x="66.04" y="7.62" rot="R180"/>
-<instance part="R16" gate="G$1" x="66.04" y="0" rot="R180"/>
 <instance part="SUPPLY9" gate="G$1" x="-76.2" y="71.12"/>
+<instance part="GND8" gate="1" x="-78.74" y="5.08"/>
+<instance part="GND14" gate="1" x="116.84" y="25.4"/>
+<instance part="GND15" gate="1" x="116.84" y="-12.7"/>
+<instance part="R13" gate="G$1" x="116.84" y="35.56" rot="R90"/>
+<instance part="R14" gate="G$1" x="116.84" y="-2.54" rot="R90"/>
+<instance part="U$2" gate="G$1" x="17.78" y="114.3"/>
 </instances>
 <busses>
@@
 <wire x1="104.14" y1="5.08" x2="111.76" y2="5.08" width="0.1524" layer="91"/>
 <pinref part="F2" gate="G$1" pin="1"/>
-<wire x1="111.76" y1="5.08" x2="119.38" y2="5.08" width="0.1524" layer="91"/>
+<wire x1="111.76" y1="5.08" x2="116.84" y2="5.08" width="0.1524" layer="91"/>
+<wire x1="116.84" y1="5.08" x2="119.38" y2="5.08" width="0.1524" layer="91"/>
+<wire x1="116.84" y1="2.54" x2="116.84" y2="5.08" width="0.1524" layer="91"/>
+<pinref part="R14" gate="G$1" pin="2"/>
 </segment>
 </net>
@@
 <wire x1="106.68" y1="43.18" x2="111.76" y2="43.18" width="0.1524" layer="91"/>
 <pinref part="F1" gate="G$1" pin="1"/>
-<wire x1="111.76" y1="43.18" x2="119.38" y2="43.18" width="0.1524" layer="91"/>
+<wire x1="111.76" y1="43.18" x2="116.84" y2="43.18" width="0.1524" layer="91"/>
+<wire x1="116.84" y1="43.18" x2="119.38" y2="43.18" width="0.1524" layer="91"/>
+<wire x1="116.84" y1="40.64" x2="116.84" y2="43.18" width="0.1524" layer="91"/>
+<pinref part="R13" gate="G$1" pin="2"/>
 </segment>
 </net>
@@
 <segment>
 <pinref part="U2" gate="G$1" pin="SDA"/>
-<wire x1="78.74" y1="10.16" x2="71.12" y2="10.16" width="0.1524" layer="91"/>
+<wire x1="78.74" y1="10.16" x2="76.2" y2="10.16" width="0.1524" layer="91"/>
 <label x="71.12" y="10.16" size="1.778" layer="95"/>
+<pinref part="U2" gate="G$1" pin="A1"/>
+<wire x1="76.2" y1="10.16" x2="71.12" y2="10.16" width="0.1524" layer="91"/>
+<wire x1="78.74" y1="5.08" x2="76.2" y2="5.08" width="0.1524" layer="91"/>
+<wire x1="76.2" y1="5.08" x2="76.2" y2="7.62" width="0.1524" layer="91"/>
+<pinref part="U2" gate="G$1" pin="A0"/>
+<wire x1="76.2" y1="7.62" x2="76.2" y2="10.16" width="0.1524" layer="91"/>
+<wire x1="78.74" y1="7.62" x2="76.2" y2="7.62" width="0.1524" layer="91"/>
 </segment>
 </net>
@@
 </segment>
 <segment>
-<pinref part="ISP1" gate="G$1" pin="VCC"/>
-<wire x1="114.3" y1="93.98" x2="124.46" y2="93.98" width="0.1524" layer="91"/>
-<pinref part="SUPPLY3" gate="G$1" pin="5V"/>
-<wire x1="124.46" y1="96.52" x2="124.46" y2="93.98" width="0.1524" layer="91"/>
-</segment>
-<segment>
 <pinref part="U1" gate="G$1" pin="VCC"/>
 <pinref part="SUPPLY5" gate="G$1" pin="5V"/>
@@
 <pinref part="GND4" gate="1" pin="GND"/>
 <wire x1="78.74" y1="40.64" x2="76.2" y2="40.64" width="0.1524" layer="91"/>
+<wire x1="76.2" y1="40.64" x2="76.2" y2="45.72" width="0.1524" layer="91"/>
+<pinref part="U1" gate="G$1" pin="A1"/>
+<wire x1="76.2" y1="45.72" x2="78.74" y2="45.72" width="0.1524" layer="91"/>
+<pinref part="U1" gate="G$1" pin="A0"/>
+<wire x1="78.74" y1="48.26" x2="76.2" y2="48.26" width="0.1524" layer="91"/>
+<wire x1="76.2" y1="48.26" x2="76.2" y2="45.72" width="0.1524" layer="91"/>
 </segment>
 <segment>
@@
 <wire x1="132.08" y1="0" x2="132.08" y2="2.54" width="0.1524" layer="91"/>
 </segment>
+<segment>
+<pinref part="GND8" gate="1" pin="GND"/>
+<pinref part="Q1" gate="G$1" pin="E"/>
+<wire x1="-78.74" y1="7.62" x2="-78.74" y2="10.16" width="0.1524" layer="91"/>
+</segment>
+<segment>
+<pinref part="GND15" gate="1" pin="GND"/>
+<wire x1="116.84" y1="-10.16" x2="116.84" y2="-7.62" width="0.1524" layer="91"/>
+<pinref part="R14" gate="G$1" pin="1"/>
+</segment>
+<segment>
+<pinref part="GND14" gate="1" pin="GND"/>
+<wire x1="116.84" y1="27.94" x2="116.84" y2="30.48" width="0.1524" layer="91"/>
+<pinref part="R13" gate="G$1" pin="1"/>
+</segment>
 </net>
 <net name="N$12" class="0">
@@
 </segment>
 </net>
-<net name="N$20" class="0">
+<net name="EN" class="0">
 <segment>
 <pinref part="JP3" gate="G$1" pin="5"/>
 <wire x1="-93.98" y1="76.2" x2="-88.9" y2="76.2" width="0.1524" layer="91"/>
+<label x="-93.98" y="76.2" size="1.778" layer="95"/>
+</segment>
+<segment>
+<pinref part="Q1" gate="G$1" pin="C"/>
+<wire x1="-78.74" y1="20.32" x2="-78.74" y2="25.4" width="0.1524" layer="91"/>
+<label x="-78.74" y="22.86" size="1.778" layer="95"/>
 </segment>
 </net>
@@
 </segment>
 </net>
-<net name="N$28" class="0">
-<segment>
-<pinref part="U1" gate="G$1" pin="A0"/>
-<pinref part="R13" gate="G$1" pin="1"/>
-<wire x1="78.74" y1="48.26" x2="71.12" y2="48.26" width="0.1524" layer="91"/>
-</segment>
-</net>
-<net name="N$29" class="0">
-<segment>
-<pinref part="U1" gate="G$1" pin="A1"/>
-<wire x1="78.74" y1="45.72" x2="71.12" y2="45.72" width="0.1524" layer="91"/>
-<pinref part="R14" gate="G$1" pin="1"/>
-<wire x1="71.12" y1="45.72" x2="71.12" y2="40.64" width="0.1524" layer="91"/>
-</segment>
-</net>
-<net name="N$30" class="0">
-<segment>
-<pinref part="U2" gate="G$1" pin="A0"/>
-<pinref part="R15" gate="G$1" pin="1"/>
-<wire x1="78.74" y1="7.62" x2="71.12" y2="7.62" width="0.1524" layer="91"/>
-</segment>
-</net>
-<net name="N$31" class="0">
-<segment>
-<pinref part="U2" gate="G$1" pin="A1"/>
-<wire x1="78.74" y1="5.08" x2="71.12" y2="5.08" width="0.1524" layer="91"/>
-<pinref part="R16" gate="G$1" pin="1"/>
-<wire x1="71.12" y1="5.08" x2="71.12" y2="0" width="0.1524" layer="91"/>
-</segment>
-</net>
+<net name="N$1" class="0">
+<segment>
+<pinref part="R8" gate="G$1" pin="1"/>
+<pinref part="Q1" gate="G$1" pin="B"/>
+<wire x1="-86.36" y1="15.24" x2="-83.82" y2="15.24" width="0.1524" layer="91"/>
+</segment>
+</net>
+<net name="N$5" class="0">
+<segment>
+<pinref part="ISP1" gate="G$1" pin="VCC"/>
+<wire x1="114.3" y1="93.98" x2="124.46" y2="93.98" width="0.1524" layer="91"/>
+<wire x1="124.46" y1="96.52" x2="124.46" y2="93.98" width="0.1524" layer="91"/>
+</segment>
+</net>
