File: Fuente.brd (EAGLE design)
At the start: 1 part, among them IC1 MEGA8-AI

Commit message: Last
Parts:
- added ISP1: AVRISP-6, adafruit:AVRISP
Connections:
- net GND: now also ISP1.6
- net VCC: now also ISP1.2
Changed lines of the file:
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@@
 <layer number="48" name="Document" color="7" fill="1" visible="yes" active="yes"/>
 <layer number="49" name="Reference" color="7" fill="1" visible="yes" active="yes"/>
+<layer number="50" name="dxf" color="7" fill="1" visible="no" active="yes"/>
 <layer number="51" name="tDocu" color="7" fill="1" visible="yes" active="yes"/>
 <layer number="52" name="bDocu" color="7" fill="1" visible="yes" active="yes"/>
+<layer number="53" name="tGND_GNDA" color="7" fill="9" visible="no" active="no"/>
+<layer number="54" name="bGND_GNDA" color="1" fill="9" visible="no" active="no"/>
+<layer number="56" name="wert" color="7" fill="1" visible="yes" active="yes"/>
 <layer number="91" name="Nets" color="2" fill="1" visible="no" active="no"/>
 <layer number="92" name="Busses" color="1" fill="1" visible="no" active="no"/>
@@
 <layer number="97" name="Info" color="7" fill="1" visible="no" active="no"/>
 <layer number="98" name="Guide" color="6" fill="1" visible="no" active="no"/>
+<layer number="100" name="Muster" color="7" fill="1" visible="no" active="no"/>
+<layer number="101" name="Patch_Top" color="12" fill="4" visible="yes" active="yes"/>
+<layer number="102" name="Vscore" color="7" fill="1" visible="yes" active="yes"/>
+<layer number="103" name="fp3" color="7" fill="1" visible="no" active="yes"/>
+<layer number="104" name="Name" color="7" fill="1" visible="yes" active="yes"/>
+<layer number="105" name="Beschreib" color="9" fill="1" visible="yes" active="yes"/>
+<layer number="106" name="BGA-Top" color="4" fill="1" visible="yes" active="yes"/>
+<layer number="107" name="BD-Top" color="5" fill="1" visible="yes" active="yes"/>
+<layer number="108" name="fp8" color="7" fill="1" visible="no" active="yes"/>
+<layer number="109" name="fp9" color="7" fill="1" visible="no" active="yes"/>
+<layer number="110" name="fp0" color="7" fill="1" visible="no" active="yes"/>
+<layer number="111" name="LPC17xx" color="7" fill="1" visible="yes" active="yes"/>
+<layer number="112" name="tSilk" color="7" fill="1" visible="yes" active="yes"/>
+<layer number="116" name="Patch_BOT" color="9" fill="4" visible="yes" active="yes"/>
+<layer number="121" name="_tsilk" color="7" fill="1" visible="yes" active="yes"/>
+<layer number="122" name="_bsilk" color="7" fill="1" visible="yes" active="yes"/>
+<layer number="123" name="tTestmark" color="7" fill="1" visible="no" active="yes"/>
+<layer number="124" name="bTestmark" color="7" fill="1" visible="no" active="yes"/>
+<layer number="125" name="_tNames" color="7" fill="1" visible="yes" active="yes"/>
+<layer number="126" name="_bNames" color="7" fill="1" visible="yes" active="yes"/>
+<layer number="127" name="_tValues" color="7" fill="1" visible="yes" active="yes"/>
+<layer number="128" name="_bValues" color="7" fill="1" visible="yes" active="yes"/>
+<layer number="131" name="tAdjust" color="7" fill="1" visible="no" active="yes"/>
+<layer number="132" name="bAdjust" color="7" fill="1" visible="no" active="yes"/>
+<layer number="144" name="Drill_legend" color="7" fill="1" visible="yes" active="yes"/>
+<layer number="151" name="HeatSink" color="7" fill="1" visible="yes" active="yes"/>
+<layer number="152" name="_bDocu" color="7" fill="1" visible="yes" active="yes"/>
+<layer number="199" name="Contour" color="7" fill="1" visible="yes" active="yes"/>
+<layer number="200" name="200bmp" color="1" fill="10" visible="yes" active="yes"/>
+<layer number="201" name="201bmp" color="2" fill="1" visible="no" active="no"/>
+<layer number="202" name="202bmp" color="3" fill="1" visible="no" active="no"/>
+<layer number="203" name="203bmp" color="4" fill="10" visible="yes" active="yes"/>
+<layer number="204" name="204bmp" color="5" fill="10" visible="yes" active="yes"/>
+<layer number="205" name="205bmp" color="6" fill="10" visible="yes" active="yes"/>
+<layer number="206" name="206bmp" color="7" fill="10" visible="yes" active="yes"/>
+<layer number="207" name="207bmp" color="8" fill="10" visible="yes" active="yes"/>
+<layer number="208" name="208bmp" color="9" fill="10" visible="yes" active="yes"/>
+<layer number="209" name="209bmp" color="7" fill="1" visible="no" active="yes"/>
+<layer number="210" name="210bmp" color="7" fill="1" visible="no" active="yes"/>
+<layer number="211" name="211bmp" color="7" fill="1" visible="yes" active="yes"/>
+<layer number="212" name="212bmp" color="7" fill="1" visible="yes" active="yes"/>
+<layer number="213" name="213bmp" color="7" fill="1" visible="yes" active="yes"/>
+<layer number="214" name="214bmp" color="7" fill="1" visible="yes" active="yes"/>
+<layer number="215" name="215bmp" color="7" fill="1" visible="yes" active="yes"/>
+<layer number="216" name="216bmp" color="7" fill="1" visible="yes" active="yes"/>
+<layer number="217" name="217bmp" color="18" fill="1" visible="no" active="no"/>
+<layer number="218" name="218bmp" color="19" fill="1" visible="no" active="no"/>
+<layer number="219" name="219bmp" color="20" fill="1" visible="no" active="no"/>
+<layer number="220" name="220bmp" color="21" fill="1" visible="no" active="no"/>
+<layer number="221" name="221bmp" color="22" fill="1" visible="no" active="no"/>
+<layer number="222" name="222bmp" color="23" fill="1" visible="no" active="no"/>
+<layer number="223" name="223bmp" color="24" fill="1" visible="no" active="no"/>
+<layer number="224" name="224bmp" color="25" fill="1" visible="no" active="no"/>
+<layer number="248" name="Housing" color="7" fill="1" visible="yes" active="yes"/>
+<layer number="249" name="Edge" color="7" fill="1" visible="yes" active="yes"/>
+<layer number="250" name="Descript" color="7" fill="1" visible="no" active="no"/>
+<layer number="251" name="SMDround" color="7" fill="1" visible="no" active="no"/>
+<layer number="254" name="cooling" color="7" fill="1" visible="yes" active="yes"/>
 </layers>
 <board>
@@
 <attribute name="OC_FARNELL" value="9171371" x="-17.78" y="-7.62" size="1.778" layer="27" display="off"/>
 </element>
+<element name="ISP1" library="adafruit" package="AVRISP" value="AVRISP-6" x="-26.67" y="-7.62"/>
 </elements>
 <signals>
@@
 <contactref element="IC1" pad="5"/>
 <contactref element="IC1" pad="21"/>
+<contactref element="ISP1" pad="6"/>
+<wire x1="-22.0726" y1="-8.02" x2="-25.4" y2="-10.16" width="0" layer="19" extent="1-1"/>
 <wire x1="-22.0726" y1="-6.42" x2="-22.0726" y2="-8.02" width="0" layer="19" extent="1-1"/>
 <wire x1="-13.4874" y1="-7.22" x2="-22.0726" y2="-8.02" width="0" layer="19" extent="1-1"/>
@@
 <contactref element="IC1" pad="4"/>
 <contactref element="IC1" pad="6"/>
-<wire x1="-22.0726" y1="-7.22" x2="-22.0726" y2="-8.82" width="0" layer="19" extent="1-1"/>
+<contactref element="ISP1" pad="2"/>
+<wire x1="-22.0726" y1="-7.22" x2="-25.4" y2="-5.08" width="0" layer="19" extent="1-1"/>
+<wire x1="-22.0726" y1="-8.82" x2="-22.0726" y2="-7.22" width="0" layer="19" extent="1-1"/>
 </signal>
 <signal name="AVCC">

Commit message: actu
Parts:
- removed IC1: MEGA8-AI, atmel:TQFP32-08
- added JP1: USBSMD, SparkFun-Connectors:USB-MINIB
- added U$1: ATMEGA32U4TQFP, SparkFun-DigitalIC:SPARKFUN-DIGITALIC_TQFP44
- moved ISP1 58.7 mm to (27.9, 14.0)
Connections:
- removed net AVCC: IC1.18
- removed net GND: IC1.21, IC1.3, IC1.5, ISP1.6
- removed net VCC: IC1.4, IC1.6, ISP1.2
- new net MISO: ISP1.1, U$1.11
- new net MOSI: ISP1.4, U$1.10
- new net N$3: ISP1.5
- new net N$4: ISP1.2
- new net N$6: ISP1.6
- new net SCK: ISP1.3, U$1.9
Changed lines of the file:
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@@
 <?xml version="1.0" encoding="utf-8"?>
 <!DOCTYPE eagle SYSTEM "eagle.dtd">
-<eagle version="6.2">
+<eagle version="6.3">
 <drawing>
 <settings>
@@
 </class>
 </classes>
-<designrules>
+<designrules name="default">
 <description language="de">&lt;b&gt;EAGLE Design Rules&lt;/b&gt;
 &lt;p&gt;
@@
 </autorouter>
 <elements>
-<element name="IC1" library="atmel" package="TQFP32-08" value="MEGA8-AI" x="-17.78" y="-7.62">
-<attribute name="OC_NEWARK" value="73M8863" x="-17.78" y="-7.62" size="1.778" layer="27" display="off"/>
-<attribute name="MPN" value="ATMEGA8-16AU" x="-17.78" y="-7.62" size="1.778" layer="27" display="off"/>
-<attribute name="MF" value="" x="-17.78" y="-7.62" size="1.778" layer="27" display="off"/>
-<attribute name="OC_FARNELL" value="9171371" x="-17.78" y="-7.62" size="1.778" layer="27" display="off"/>
-</element>
-<element name="ISP1" library="adafruit" package="AVRISP" value="AVRISP-6" x="-26.67" y="-7.62"/>
+<element name="ISP1" library="adafruit" package="AVRISP" value="AVRISP-6" x="27.94" y="13.97"/>
+<element name="U$1" library="SparkFun-DigitalIC" package="SPARKFUN-DIGITALIC_TQFP44" value="ATMEGA32U4TQFP" x="30.48" y="2.54"/>
+<element name="JP1" library="SparkFun-Connectors" package="USB-MINIB" value="USBSMD" x="19.05" y="2.54"/>
 </elements>
 <signals>
-<signal name="GND">
-<contactref element="IC1" pad="3"/>
-<contactref element="IC1" pad="5"/>
-<contactref element="IC1" pad="21"/>
+<signal name="MISO">
+<contactref element="ISP1" pad="1"/>
+<contactref element="U$1" pad="11"/>
+<wire x1="24.68" y1="-1.46" x2="26.67" y2="16.51" width="0" layer="19" extent="1-1"/>
+</signal>
+<signal name="SCK">
+<contactref element="ISP1" pad="3"/>
+<contactref element="U$1" pad="9"/>
+<wire x1="24.68" y1="0.14" x2="26.67" y2="13.97" width="0" layer="19" extent="1-1"/>
+</signal>
+<signal name="N$3">
+<contactref element="ISP1" pad="5"/>
+</signal>
+<signal name="N$4">
+<contactref element="ISP1" pad="2"/>
+</signal>
+<signal name="MOSI">
+<contactref element="ISP1" pad="4"/>
+<contactref element="U$1" pad="10"/>
+<wire x1="24.68" y1="-0.66" x2="29.21" y2="13.97" width="0" layer="19" extent="1-1"/>
+</signal>
+<signal name="N$6">
 <contactref element="ISP1" pad="6"/>
-<wire x1="-22.0726" y1="-8.02" x2="-25.4" y2="-10.16" width="0" layer="19" extent="1-1"/>
-<wire x1="-22.0726" y1="-6.42" x2="-22.0726" y2="-8.02" width="0" layer="19" extent="1-1"/>
-<wire x1="-13.4874" y1="-7.22" x2="-22.0726" y2="-8.02" width="0" layer="19" extent="1-1"/>
-</signal>
-<signal name="VCC">
-<contactref element="IC1" pad="4"/>
-<contactref element="IC1" pad="6"/>
-<contactref element="ISP1" pad="2"/>
-<wire x1="-22.0726" y1="-7.22" x2="-25.4" y2="-5.08" width="0" layer="19" extent="1-1"/>
-<wire x1="-22.0726" y1="-8.82" x2="-22.0726" y2="-7.22" width="0" layer="19" extent="1-1"/>
-</signal>
-<signal name="AVCC">
-<contactref element="IC1" pad="18"/>
 </signal>
 </signals>

Commit message: Sch updated
Parts:
- added C1: 10uF, SparkFun-Capacitors:CPOL-RADIAL-10UF-25V
- added F1, F2: (no value), adafruit:1812
- added Q1: (no value), SparkFun-DiscreteSemi:SOT23
- added R1, R2, R7, R9: 10k, adafruit:M0805
- added R10, R11, R12: 220, SparkFun-Resistors:0805
- added R3, R4: .1, adafruit:R2512
- added R5, R6: 22, adafruit:0309/12
- added R8: 1k, adafruit:M0805
- added S1, S5: 50-2POLE30, switch:50-2POLE30
- added S2: 75CF36-2, switch:75CF36-2
- added S3: (no value), switch:CK102X06
- added S4, S6: ELMA-01-2X6, switch:ELMA-01-2X6
- added S7, S8: SWITCH-MOMENTARY-212MM, SparkFun-Electromechanical:TACTILE-PTH-12MM
- added U$2, U$3: (no value), SparkFun-Electromechanical:POT_ALPHA_RV16AF-20
- added U$4: LED-TRICOLOR, SparkFun-LED:LED-TRICOLOR-SMD
- added U1, U2: (no value), microbuilder:SOT23-8
- added Y1: (no value), SparkFun-FreqCtrl:RESONATOR-PTH
- moved U$1 13.1 mm to (41.9, 8.89)
- moved JP1 7.41 mm to (15.2, 8.89)
Connections:
- new net 5V: ISP1.2, R1.2, R2.2, R7.2, U$1.14, U$1.2, U$1.24, U$1.34, U$1.44, U$4.A, U1.4, U2.4
- new net GND: C1.2, ISP1.6, JP1.GND, R9.2, S7.3, U$1.15, U$1.23, U$1.35, U$1.43, U$1.5, U1.3, U2.3, Y1.2
- new net N$1: R4.2, U2.1
- new net N$10: R6.2, U$1.3
- new net N$11: JP1.D-, R6.1
- new net N$12: U$1.17, Y1.1
- new net N$13: U$1.16, Y1.3
- new net N$14: R11.2, U$4.B
- new net N$15: R12.2, U$4.G
- new net N$2: F2.1, R4.1, U2.2
- new net N$5: R3.2, U1.1
- new net N$7: F1.1, R3.1, U1.2
- new net N$8: JP1.D+, R5.1
- new net N$9: R5.2, U$1.4
- new net R1: ISP1.5, R7.1, S7.1, U$1.13
- new net SCL: R2.1, U$1.18, U1.5, U2.5
- new net SDA: R1.1, U$1.19, U1.6, U2.6
- net N$3: now also C1.1, JP1.VBUS, U$1.7; no longer ISP1.5
- net N$4: now also R9.1, U$1.33; no longer ISP1.2
- net N$6: now also R10.2, U$4.R; no longer ISP1.6

Commit message: Sch and Pcb updated
Parts:
- removed S1, S5: 50-2POLE30, switch:50-2POLE30
- removed S2: 75CF36-2, switch:75CF36-2
- removed S3: (no value), switch:CK102X06
- removed S4, S6: ELMA-01-2X6, switch:ELMA-01-2X6
- added JP2, JP3: (no value), SparkFun-Connectors:1X08_LONGPADS
- added JP4, JP5: (no value), SparkFun-Connectors:1X02_LOCK_LONGPADS
- added R13, R14, R15, R16: 10k, adafruit:M0805
- moved R12 111.0 mm to (57.2, 29.4)
- moved R11 108.0 mm to (57.2, 31.4)
- moved R10 103.1 mm to (57.2, 27.4)
- moved R9 99.1 mm to (54.6, 36.8)
- moved U$4 95.8 mm to (61.0, 29.2)
- moved C1 92.7 mm to (48.3, 44.5)
- moved U$2 82.7 mm to (78.0, 1.55)
- moved U$3 80.3 mm to (57.7, 1.55)
- moved F1 75.2 mm to (78.0, 61.7)
- moved U2 74.7 mm to (61.0, 72.0), turned to 90 degrees
- moved R5 74.3 mm to (20.3, 70.8)
- moved S8 67.3 mm to (91.4, 31.8)
- moved R6 65.7 mm to (20.3, 74.5)
- moved JP1 64.6 mm to (5.40, 72.8)
- moved U$1 64.1 mm to (37.8, 72.8)
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Connections:
- removed net N$1: R4.2, U2.1
- removed net N$5: R3.2, U1.1
- new net INV12: JP2.7, JP2.8, JP3.8
- new net INV33: JP2.3, JP2.4, JP3.6
- new net INV5: JP2.5, JP2.6, JP3.7
- new net N$16: F1.2, JP4.2
- new net N$17: F2.2, JP5.2
- new net N$19: JP3.4
- new net N$20: JP3.5
- new net N$28: R13.1, U1.7
- new net N$29: R14.1, U1.8
- new net N$30: R15.1, U2.7
- new net N$31: R16.1, U2.8
- new net V1: JP2.1, R3.2, U1.1
- new net V2: JP2.2, R4.2, U2.1
- net 5V: now also JP3.3
- net GND: now also JP3.1, JP3.2, JP4.1, JP5.1
Routing:
- net V2: track 0.00 -> 150.1 mm
- net V1: track 0.00 -> 123.6 mm
- net INV33: track 0.00 -> 95.5 mm
- net INV5: track 0.00 -> 71.3 mm
- net INV12: track 0.00 -> 42.0 mm
- net N$9: track 0.00 -> 6.88 mm
- net N$8: track 0.00 -> 6.87 mm
- net N$11: track 0.00 -> 6.43 mm
- net N$10: track 0.00 -> 5.68 mm
- net N$14: track 0.00 -> 5.54 mm
- net N$12: track 0.00 -> 4.22 mm
- net N$13: track 0.00 -> 4.20 mm
- net N$7: track 0.00 -> 3.15 mm
- net N$2: track 0.00 -> 3.15 mm
- net N$15: track 0.00 -> 2.73 mm
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Other:
- board outline added: 100 x 100 mm

Commit message: pcb and sch updated
Parts:
- moved JP3 17.1 mm to (27.9, 29.2)
- moved JP2 15.3 mm to (49.5, 19.1)
- moved ISP1 14.5 mm to (25.4, 61.0)
- moved JP5 12.1 mm to (74.0, 65.0)
- moved JP4 11.2 mm to (74.0, 60.1), turned to 270 degrees
- moved F2 11.2 mm to (67.7, 67.7)
- moved F1 11.2 mm to (67.7, 57.4)
- moved R4 11.2 mm to (59.7, 67.7)
- moved U2 11.2 mm to (50.7, 67.7)
- moved R3 11.2 mm to (59.7, 57.4)
- moved U1 11.2 mm to (50.7, 57.4)
- moved U$3 7.62 mm to (65.3, 1.55)
- moved U$2 5.08 mm to (83.1, 1.55)
- moved Y1 2.54 mm to (37.4, 61.2)
- moved JP1 1.31 mm to (4.74, 73.9)
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Routing:
- net V2: track 150.1 -> 5.30 mm
- net V1: track 123.6 -> 5.30 mm
- net N$7: track 3.15 -> 17.9 mm
- net N$2: track 3.15 -> 17.7 mm
- net INV33: track 95.5 -> 89.5 mm
- net INV5: track 71.3 -> 66.0 mm
- net INV12: track 42.0 -> 36.7 mm
- net N$12: track 4.22 -> 0.00 mm
- net N$13: track 4.20 -> 0.00 mm
- net N$9: track 6.88 -> 6.08 mm
- net N$11: track 6.43 -> 7.14 mm
- net N$8: track 6.87 -> 7.47 mm
Other:
- board size 100 x 100 mm -> 100 x 100.2 mm

Commit message: pcb and sch updated
Parts:
- removed R15, R16: 10k, adafruit:M0805
- R13, R14: value 10k -> 1M
- U$2: value (none) -> M08X2; device SparkFun-Electromechanical:POT_ALPHA_RV16AF-20 -> SparkFun-Connectors:2X8
- moved U$2 74.1 mm to (35.6, 58.4), turned to 90 degrees
- moved Q1 45.5 mm to (33.6, 38.9), turned to 90 degrees
- moved C1 44.9 mm to (78.7, 11.4)
- moved Y1 37.0 mm to (51.4, 26.9)
- moved U$1 34.5 mm to (48.0, 39.8)
- moved ISP1 30.3 mm to (36.8, 32.8)
- moved R7 24.4 mm to (43.2, 29.2)
- moved R14 22.2 mm to (70.7, 66.4), turned to 180 degrees
- moved R8 21.6 mm to (38.1, 39.4)
- moved U$4 21.2 mm to (79.8, 19.5)
- moved R10 21.2 mm to (76.0, 17.7)
- moved R11 21.2 mm to (76.0, 21.7)
- moved R12 21.2 mm to (76.0, 19.7)
- moved R2 17.8 mm to (72.4, 40.6)
- moved R9 16.5 mm to (69.8, 30.5)
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Connections:
- removed net N$20: JP3.5
- removed net N$28: R13.1, U1.7
- removed net N$29: R14.1, U1.8
- removed net N$30: R15.1, U2.7
- removed net N$31: R16.1, U2.8
- new net EN: JP3.5, Q1.3
- new net N$1: Q1.1, R8.1
- new net N$5: ISP1.2
- net 5V: no longer ISP1.2
- net GND: now also Q1.2, R13.1, R14.1, U1.7, U1.8
- net N$2: now also R14.2
- net N$7: now also R13.2
- net SDA: now also U2.7, U2.8
Routing:
- net INV33: track 89.5 -> 2.54 mm
- net INV5: track 66.0 -> 2.54 mm
- net N$10: track 5.51 -> 40.8 mm
- net INV12: track 36.7 -> 2.54 mm
- net N$9: track 6.08 -> 38.4 mm
- net SCL: track 0.00 -> 15.8 mm
- net SDA: track 0.00 -> 15.4 mm
- net GND: track 0.00 -> 14.2 mm
- net N$12: track 0.00 -> 11.4 mm
- net R1: track 0.00 -> 10.2 mm
- net N$13: track 0.00 -> 7.83 mm
- net N$16: track 0.00 -> 4.24 mm
- net N$17: track 0.00 -> 4.24 mm
- net SCK: track 0.00 -> 3.56 mm
- net N$2: track 17.7 -> 14.4 mm
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Other:
- outline, holes or cut-outs redrawn

Commit message: pcb and sch updated
Parts:
- removed U$2: M08X2, SparkFun-Connectors:2X8
- added C2, C3: 1u, adafruit:E2,5-6
- added C4: 100n, adafruit:C0805K
- added Q2: (no value), SparkFun-DiscreteSemi:SOT23
- added R15: (no value), pot:CT6
- added R16: 1k, adafruit:M0805
- added U3: LCD-16X28X2, SparkFun-Displays:LCD-8X2
- moved C1 24.8 mm to (62.2, 29.9), turned to 180 degrees
- moved R9 18.0 mm to (59.9, 45.5), turned to 90 degrees
- moved U$4 14.9 mm to (80.0, 4.69), turned to 270 degrees
- moved R11 14.6 mm to (82.2, 8.46), turned to 270 degrees
- moved R12 12.0 mm to (80.2, 8.46), turned to 270 degrees
- moved R8 9.61 mm to (32.8, 31.4)
- moved R10 9.48 mm to (78.2, 8.46), turned to 270 degrees
- moved R7 7.81 mm to (48.2, 23.2)
- moved ISP1 6.52 mm to (42.3, 29.3)
- moved R1 4.30 mm to (71.1, 44.1), turned to 180 degrees
- moved U$1 4.12 mm to (52.0, 38.8)
- moved Q1 4.00 mm to (33.6, 34.9)
- moved R2 3.91 mm to (75.4, 43.1)
- moved S7 3.00 mm to (91.4, 16.1)
- moved R5 2.54 mm to (17.8, 72.0)
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Connections:
- new net B: R11.1, U$1.28
- new net BTN: S8.3, U$1.29
- new net CTRL: U$1.25, U$3.2
- new net DB4: U$1.39, U3.11
- new net DB5: U$1.38, U3.12
- new net DB6: U$1.37, U3.13
- new net DB7: U$1.36, U3.14
- new net E: U$1.40, U3.6
- new net G: R12.1, U$1.27
- new net LUZ: R16.2, U$1.1
- new net N$18: C4.1, U$1.42
- new net N$21: R15.S, U3.3
- new net N$22: C2.+, U$1.6
- new net N$29: Q2.3, U3.16
- new net ON: R8.2, U$1.8
- new net R: R10.1, U$1.26
- new net RS: U$1.41, U3.4
- net 5V: now also C3.+, JP3.4, R15.A, U$3.3, U3.15, U3.2; no longer JP3.3
- net GND: now also C2.-, C3.-, C4.2, JP3.3, Q2.2, R15.E, S7.1, S8.1, U$3.1, U3.1, U3.10, U3.5, U3.7, U3.8, U3.9; no longer S7.3
- net N$19: now also Q2.1, R16.1; no longer JP3.4
- net R1: now also S7.3; no longer S7.1
Routing:
- net V2: track 7.30 -> 162.7 mm
- net V1: track 4.70 -> 137.8 mm
- net GND: track 14.2 -> 127.1 mm, vias 0 -> 5
- net INV33: track 2.54 -> 101.6 mm
- net N$3: track 0.00 -> 75.3 mm
- net INV5: track 2.54 -> 75.1 mm
- net LUZ: track 0.00 -> 65.4 mm
- net R1: track 10.2 -> 61.9 mm
- net 5V: track 0.01 -> 47.0 mm, vias 1 -> 3
- net B: track 0.00 -> 41.9 mm
- net SDA: track 15.4 -> 56.1 mm
- net RS: track 0.00 -> 40.3 mm
- net G: track 0.00 -> 39.8 mm
- net E: track 0.00 -> 39.4 mm
- net R: track 0.00 -> 37.7 mm
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
Commit message: updated pcb and sch
ready for first print
Parts:
- moved C1 62.6 mm to (11.7, 66.9), turned to 270 degrees
- moved R1 20.1 mm to (63.5, 25.5), turned to 90 degrees
- moved R2 20.0 mm to (66.0, 25.5), turned to 90 degrees
- moved R7 17.7 mm to (32.2, 30.7), turned to 180 degrees
- moved C3 14.5 mm to (75.0, 33.0)
- moved R8 6.80 mm to (38.3, 35.4)
- moved U$3 2.00 mm to (64.1, 3.55)
- moved Y1 1.41 mm to (54.7, 25.9)
- moved ISP1 1.00 mm to (42.3, 30.3)
- moved Q1 0.99 mm to (34.3, 34.3), turned to 180 degrees
Routing:
- net GND: track 127.1 -> 577.2 mm, vias 5 -> 20
- net 5V: track 47.0 -> 315.1 mm, vias 3 -> 16
- net R1: track 61.9 -> 115.5 mm, vias 0 -> 3
- net CTRL: track 0.00 -> 45.3 mm
- net SCL: track 39.7 -> 75.9 mm, vias 0 -> 2
- net SDA: track 56.1 -> 83.8 mm, vias 0 -> 2
- net N$24: track 0.00 -> 13.5 mm, vias 1 -> 0
- net EN: track 0.00 -> 9.91 mm
- net N$20: track 0.00 -> 9.57 mm, vias 1 -> 0
- net MOSI: track 0.00 -> 9.22 mm
- net SCK: track 0.00 -> 7.74 mm
- net ON: track 0.00 -> 7.73 mm
- net N$13: track 0.01 -> 7.55 mm
- net N$12: track 3.85 -> 10.6 mm
- net N$23: track 0.00 -> 6.41 mm, vias 1 -> 0
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- added copper zone on layer 1, net 5V
- added copper zone on layer 1, net GND
Other:
- board size 100 x 100.2 mm -> 100 x 100 mm
- board text added: "Ch9FOD 2012"
